File: projet-Kicad/projet-v1/projet-v1.kicad_pcb (KiCad board)
At the start: 2 copper layers, 68.6 x 53.3 mm, 8 parts, among them J1 Power, J2 Digital/PWM, J3 Analog, J4 Digital/PWM

Commit message: MAJ projet Kicad version envoyée à Cathy
Parts:
- added C1: 100n, Capacitor_THT:C_Disc_D4.7mm_W2.5mm_P5.00mm, F.Cu at (124.0, 68.5)
- added C2: 100n, Capacitor_THT:C_Disc_D4.7mm_W2.5mm_P5.00mm, F.Cu at (143.0, 86.2)
- added C4: 1u, Capacitor_THT:C_Rect_L7.0mm_W4.5mm_P5.00mm, F.Cu at (135.0, 79.0)
- added C5: 100n, Capacitor_THT:C_Disc_D4.7mm_W2.5mm_P5.00mm, F.Cu at (144.0, 53.0)
- added R1: 100k, Resistor_THT:R_Axial_DIN0207_L6.3mm_D2.5mm_P5.08mm_Vertical, F.Cu at (129.5, 68.7)
- added R3: 100k, Resistor_THT:R_Axial_DIN0207_L6.3mm_D2.5mm_P5.08mm_Vertical, F.Cu at (125.8, 90.5)
- added R4: 10k, Resistor_THT:R_Axial_DIN0207_L6.3mm_D2.5mm_P5.08mm_Vertical, F.Cu at (134.8, 83.2)
- added R5: 1k, Resistor_THT:R_Axial_DIN0207_L6.3mm_D2.5mm_P5.08mm_Vertical, F.Cu at (143.0, 72.9)
- added R6: 47k, Resistor_THT:R_Axial_DIN0207_L6.3mm_D2.5mm_P5.08mm_Vertical, F.Cu at (166.0, 80.2)
- added U1: ~, librairie-empreintes:HC05-05, F.Cu at (155.6, 75.0)
- added U2: ~, librairie-empreintes:OLED01, F.Cu at (116.0, 76.7)
- added U3: ~, librairie-empreintes:graphite-sensor, F.Cu at (138.5, 88.5)
- added U4: ~, librairie-empreintes:MCP41050, F.Cu at (131.2, 60.7)
- added U5: ~, librairie-empreintes:flex-sensor, F.Cu at (157.5, 90.0)
- added U6: ~, librairie-empreintes:KY-040, F.Cu at (161.8, 61.5)
- added U7: ~, librairie-empreintes:LTC1050, F.Cu at (125.5, 83.0)
Connections:
- net /SCL/A5 renamed SCL
- net /SDA/A4 renamed SDA
- J2 pad 10: /8 -> TXD
- J2 pad 5: /13 -> SCK
- J2 pad 7: /*11 -> SDI
- J2 pad 8: /*10 -> CS
- J2 pad 9: /*9 -> RXD
- J3 pad 1: /A0 -> ADC
- J3 pad 2: /A1 -> FS
- J4 pad 4: /4 -> SW
- J4 pad 5: /*3 -> DT
- J4 pad 6: /2 -> CLK
Routing:
- net +5V: track 0.00 -> 143.4 mm
- net Net-(U7-OUT): track 0.00 -> 61.6 mm
- net Net-(U7-+): track 0.00 -> 51.4 mm
- net R2: track 0.00 -> 41.6 mm
- net RXD: track 0.00 -> 36.3 mm
- net TXD: track 0.00 -> 34.9 mm
- net CLK: track 0.00 -> 32.7 mm
- net SCL: track 0.00 -> 32.6 mm
- net SDA: track 0.00 -> 32.1 mm
- net ADC: track 0.00 -> 31.7 mm
- net FS: track 0.00 -> 30.9 mm
- net SW: track 0.00 -> 16.9 mm
- net GND: track 0.00 -> 15.1 mm
- net DT: track 0.00 -> 14.0 mm
- net SDI: track 0.00 -> 9.48 mm
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- added copper zone on B.Cu, net GND
Other:
- board text added: "Margot HERNANDEZ Esther BOIRON 4A GP"
