File: projet-Kicad/projet-v1/projet-v1.kicad_pcb (KiCad board)
At the start: 2 copper layers, 68.6 x 53.3 mm, 24 parts, among them J1 Power, J2 Digital/PWM, J3 Analog, J4 Digital/PWM

Commit message: MAJ Kicad
Parts:
- moved R6 9.01 mm to (161.0, 87.7)
- moved U5 4.51 mm to (153.2, 91.5), turned to -90 degrees
- moved R1 1.31 mm to (128.2, 68.7)
Routing:
- net FS: track 30.9 -> 12.5 mm
- net SDA: track 32.1 -> 25.9 mm
- net RXD: track 36.3 -> 32.6 mm
- net CLK: track 32.7 -> 29.0 mm
- net SCL: track 32.6 -> 29.4 mm
- net TXD: track 34.9 -> 32.6 mm
- net R2: track 41.6 -> 43.3 mm
- net +5V: track 143.4 -> 145.0 mm
- net Net-(U7-OUT): track 61.6 -> 60.3 mm
- net Net-(U7-+): track 51.4 -> 50.1 mm
- net DT: track 14.0 -> 12.9 mm
